File: DataSliceHW/DataSliceHW.kicad_sch (KiCad schematic)
At the start: 97 parts, among them SW1 SKRPABE010, SW10 SKRPABE010, SW11 SKRPABE010, SW12 SKRPABE010, SW13 SKRPABE010, SW14 SKRPABE010, SW15 SKRPABE010, SW16 SKRPABE010, SW17 SKRPABE010, SW18 SKRPABE010, SW19 SKRPABE010, SW2 SKRPABE010, SW20 SKRPABE010, SW21 SKRPABE010, SW22 SKRPABE010, SW23 SKRPABE010, SW24 SKRPABE010, SW25 SKRPABE010, SW26 SKRPABE010, SW27 SKRPABE010, SW28 SKRPABE010, SW29 SKRPABE010, SW3 SKRPABE010, SW30 SKRPABE010, SW31 SKRPABE010, SW32 SKRPABE010, SW33 SKRPABE010, SW34 SKRPABE010, SW35 SKRPABE010, SW36 SKRPABE010, SW37 SKRPABE010, SW38 SKRPABE010, SW39 SKRPABE010, SW4 SKRPABE010, SW40 SKRPABE010, SW41 SKRPABE010, SW42 SKRPABE010, SW43 SKRPABE010, SW44 SKRPABE010, SW45 SKRPABE010, SW46 SKRPABE010, SW47 SKRPABE010, SW48 SKRPABE010, SW5 SKRPABE010, SW6 SKRPABE010, SW7 SKRPABE010, SW8 SKRPABE010, SW9 SKRPABE010, U1 ESP32-C6-WROOM-1-N4

Commit message: Schematic and PCB progress Changed ESP module to S3 Added Battery outline Added Program buttons, Auto Program schematic, USB-UART without USB-C socket, SD card socket Finished: ESP, Buttons, Programming, SD card TODO: ESP USB UART, OLED, Power/Battery, USB Host, CC1101, LoRa, Ext RS232, Ext SPI
Parts:
- removed U1: ESP32-C6-WROOM-1-N4, MOD28_ESP32-C6-WROOM-1_EXP, symbol DataSlice:ESP32-C6-WROOM-1-N4
- added C1, C7: 10uF/16V(10%), Capacitor_SMD:C_0603_1608Metric_Pad1.08x0.95mm_HandSolder, symbol Device:C_Small
- added C2, C3, C8: 100nF/16V(10%), Capacitor_SMD:C_0603_1608Metric_Pad1.08x0.95mm_HandSolder, symbol Device:C_Small
- added C4, C5, C6: 1uF/16V(10%), Capacitor_SMD:C_0603_1608Metric_Pad1.08x0.95mm_HandSolder, symbol Device:C_Small
- added C9: 4.7uF/16V(10%), Capacitor_SMD:C_0603_1608Metric_Pad1.08x0.95mm_HandSolder, symbol Device:C_Small
- added J1: Micro_SD_Card_Det2, Connector_Card:microSD_HC_Hirose_DM3D-SF, symbol Connector:Micro_SD_Card_Det2
- added Q1: BC847BDW1, Package_TO_SOT_SMD:SOT-363_SC-70-6, symbol Transistor_BJT:BC847BDW1
- added R1: 1K(1%), Resistor_SMD:R_0603_1608Metric_Pad0.98x0.95mm_HandSolder, symbol Device:R_Small
- added R2: 24K(1%), Resistor_SMD:R_0603_1608Metric_Pad0.98x0.95mm_HandSolder, symbol Device:R_Small
- added R3: 47K(1%), Resistor_SMD:R_0603_1608Metric_Pad0.98x0.95mm_HandSolder, symbol Device:R_Small
- added R4, R5, R7, R8: 10K(1%), Resistor_SMD:R_0603_1608Metric_Pad0.98x0.95mm_HandSolder, symbol Device:R_Small
- added R6: 10K(1%)(NC), Resistor_SMD:R_0603_1608Metric_Pad0.98x0.95mm_HandSolder, symbol Device:R_Small
- added SW49, SW50: SKRKAHE020, Button_Switch_SMD:SW_Push_SPST_NO_Alps_SKRK, symbol Switch:SW_Push
- added U1: ESP32-S3-WROOM-1, RF_Module:ESP32-S3-WROOM-1, symbol RF_Module:ESP32-S3-WROOM-1
- added U2: CP2102N-Axx-xQFN28, Package_DFN_QFN:QFN-28-1EP_5x5mm_P0.5mm_EP3.35x3.35mm, symbol Interface_USB:CP2102N-Axx-xQFN28
- renumbered D37 to D10, D41 to D11, D45 to D12, D2 to D13, D6 to D14, D10 to D15, D14 to D16, D18 to D17, D22 to D18, D26 to D19, D5 to D2, D30 to D20, D34 to D21, D38 to D22, D42 to D23, D46 to D24, D3 to D25, D7 to D26, D11 to D27, D15 to D28, D19 to D29, D9 to D3, D23 to D30, D27 to D31, D31 to D32, D35 to D33, D39 to D34, D43 to D35, D47 to D36, D4 to D37, D8 to D38, D12 to D39, D13 to D4, D16 to D40, D20 to D41, D24 to D42, D28 to D43, D32 to D44, D36 to D45, D40 to D46, D44 to D47, D17 to D5, D21 to D6, D25 to D7, D29 to D8, D33 to D9, SW37 to SW10, SW41 to SW11, SW45 to SW12, SW2 to SW13, SW6 to SW14, SW10 to SW15, SW14 to SW16, SW18 to SW17, SW22 to SW18, SW26 to SW19, SW5 to SW2, SW30 to SW20, SW34 to SW21, SW38 to SW22, SW42 to SW23, SW46 to SW24, SW3 to SW25, SW7 to SW26, SW11 to SW27, SW15 to SW28, SW19 to SW29, SW9 to SW3, SW23 to SW30, SW27 to SW31, SW31 to SW32, SW35 to SW33, SW39 to SW34, SW43 to SW35, SW47 to SW36, SW4 to SW37, SW8 to SW38, SW12 to SW39, SW13 to SW4, SW16 to SW40, SW20 to SW41, SW24 to SW42, SW28 to SW43, SW32 to SW44, SW36 to SW45, SW40 to SW46, SW44 to SW47, SW17 to SW5, SW21 to SW6, SW25 to SW7, SW29 to SW8, SW33 to SW9
Connections:
- net Col1 renamed KB_C_0
- net KB_C_0: now also U1.39 (IO1)
- net Col10 renamed KB_C_9
- net KB_C_9: now also U1.22 (IO14)
- net Col11 renamed KB_C_10
- net KB_C_10: now also U1.8 (IO15)
- net Col12 renamed KB_C_11
- net KB_C_11: now also U1.9 (IO16)
- net Col2 renamed KB_C_1
- net KB_C_1: now also U1.38 (IO2)
- net Col3 renamed KB_C_2
- net KB_C_2: now also U1.15 (IO3)
- net Col4 renamed KB_C_3
- net KB_C_3: now also U1.4 (IO4)
- net Col5 renamed KB_C_4
- net KB_C_4: now also U1.5 (IO5)
- net Col6 renamed KB_C_5
- net KB_C_5: now also U1.6 (IO6)
- net Col7 renamed KB_C_6
- net KB_C_6: now also U1.7 (IO7)
- net Col8 renamed KB_C_7
- net KB_C_7: now also U1.12 (IO8)
- net Col9 renamed KB_C_8
- net KB_C_8: now also U1.17 (IO9)
- net Row1 renamed KB_R_0
- net KB_R_0: now also U1.26 (IO45)
- net Row2 renamed KB_R_1
- net KB_R_1: now also U1.16 (IO46)
- net Row3 renamed KB_R_2
- net KB_R_2: now also U1.24 (IO47)
- net Row4 renamed KB_R_3
- net KB_R_3: now also U1.25 (IO48)
- new net: Q1.2 (B1), R7.1
- new net: Q1.5 (B2), R8.1
- new net: C4.1, R2.2, R3.1, U2.8 (VBUS)
- new net: R1.2, U2.9 (~{RST})
- new net: R6.1, U2.11 (~{SUSPEND})
- new net DTR: Q1.1 (E1), R8.2, U2.28 (~{DTR})
- new net ESP_EN: C6.1, C9.1, Q1.3 (C2), R5.2, SW50.1, U1.3 (EN)
- new net GND: C1.1, C2.2, C3.2, C4.2, C5.2, C6.2, C7.1, C8.2, C9.2, J1.10 (DET_A), J1.11 (SHIELD), J1.6 (VSS), J1.9 (DET_B), R3.2, R6.2, SW49.2, SW50.2, U1.1 (GND), U1.40 (GND), U1.41 (GND), U2.29 (GND), U2.3 (GND)
- new net GPIO0: C5.1, Q1.6 (C1), R4.2, SW49.1, U1.27 (IO0)
- new net HOST_DN: U1.13 (USB_D-)
- new net HOST_DP: U1.14 (USB_D+)
- new net PC_DN: U2.5 (D-)
- new net PC_DP: U2.4 (D+)
- new net PC_VBUS: R2.1
- new net RS_RX: U1.11 (IO18)
- new net RS_TX: U1.10 (IO17)
- new net RTS: Q1.4 (E2), R7.2, U2.24 (~{RTS})
- new net SD_CLK: J1.5 (CLK), U1.23 (IO21)
- new net SD_CMD: J1.3 (CMD), U1.31 (IO38)
- new net SD_D0: J1.7 (DAT0), U1.32 (IO39)
- new net SD_D1: J1.8 (DAT1), U1.33 (IO40)
- new net SD_D2: J1.1 (DAT2), U1.34 (IO41)
- new net SD_D3: J1.2 (DAT3/CD), U1.35 (IO42)
- new net SPI_CK: U1.20 (IO12)
- new net SPI_CS: U1.18 (IO10)
- new net SPI_DI: U1.19 (IO11)
- new net SPI_DO: U1.21 (IO13)
- new net UART_RX: U1.36 (RXD0), U2.26 (TXD)
- new net UART_TX: U1.37 (TXD0), U2.25 (RXD)
- new net VCC: C1.2, C2.1, C3.1, C7.2, C8.1, J1.4 (VDD), R1.1, R4.1, R5.1, U1.2 (3V3), U2.6 (VDD), U2.7 (VREGIN)
- no-connect marks 0 -> 18

Commit message: Pin adjustments for SD Add display ribbon cable hole
Parts:
- added R9: 10K(1%), Resistor_SMD:R_0603_1608Metric_Pad0.98x0.95mm_HandSolder, symbol Device:R_Small
Connections:
- net VCC: now also R9.1
- net SD_D1: no longer names the net of U1.33 (IO40)
- net SD_D1: no longer J1.8 (DAT1)
- net SD_D2: no longer names the net of J1.1 (DAT2)
- net SD_D2: no longer U1.34 (IO41)
- net SD_D3: no longer names the net of J1.2 (DAT3/CD)
- net SD_D3: now also R9.2; no longer U1.35 (IO42)
- new net I2C_SCL: U1.35 (IO42)
- new net I2C_SDA: U1.34 (IO41)
- no-connect marks 18 -> 20
Other:
- moved on the sheet: C3, C4, C5, C6, C7, C8, C9, J1, Q1A, Q1B, R1, R2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

Commit message: Added OLED schematic
Parts:
- added C10, C11: 22uF/50V(10%), Capacitor_SMD:C_0603_1608Metric_Pad1.08x0.95mm_HandSolder, symbol Device:C_Small
- added C12, C9: 4.7uF/50V(10%), Capacitor_SMD:C_0402_1005Metric_Pad0.74x0.62mm_HandSolder, symbol Device:C_Small
- added C5: 4.7uF/16V(10%), Capacitor_SMD:C_0402_1005Metric_Pad0.74x0.62mm_HandSolder, symbol Device:C_Small
- added C8: 100nF/16V(10%), Capacitor_SMD:C_0402_1005Metric_Pad0.74x0.62mm_HandSolder, symbol Device:C_Small
- added D49: SS14, Diode_SMD:D_SMA_Handsoldering, symbol Device:D_Small_Filled
- added J2: 6871XX183622_687124183622, DataSlice:687124183622, symbol DataSlice:6871XX183622_687124183622
- added L1: 4.7uH, Inductor_SMD:L_Coilcraft_LPS4018, symbol Device:L_Iron_Small
- added R10: 200K(1%), Resistor_SMD:R_0402_1005Metric_Pad0.72x0.64mm_HandSolder, symbol Device:R_Small
- added R11, R4: 10K(1%), Resistor_SMD:R_0402_1005Metric_Pad0.72x0.64mm_HandSolder, symbol Device:R_Small
- added R7, R8: 4.7K(1%), Resistor_SMD:R_0402_1005Metric_Pad0.72x0.64mm_HandSolder, symbol Device:R_Small
- added R9: 1M(1%), Resistor_SMD:R_0402_1005Metric_Pad0.72x0.64mm_HandSolder, symbol Device:R_Small
- added U3: MT3608/SX1308, Package_TO_SOT_SMD:SOT-23-6_Handsoldering, symbol Regulator_Switching:MT3608
- C1, C2: footprint Capacitor_SMD:C_0603_1608Metric_Pad1.08x0.95mm_HandSolder -> Capacitor_SMD:C_0402_1005Metric_Pad0.74x0.62mm_HandSolder
- C13: renamed from C5; footprint Capacitor_SMD:C_0603_1608Metric_Pad1.08x0.95mm_HandSolder -> Capacitor_SMD:C_0402_1005Metric_Pad0.74x0.62mm_HandSolder
- C14: renamed from C6; footprint Capacitor_SMD:C_0603_1608Metric_Pad1.08x0.95mm_HandSolder -> Capacitor_SMD:C_0402_1005Metric_Pad0.74x0.62mm_HandSolder
- C15: renamed from C9; footprint Capacitor_SMD:C_0603_1608Metric_Pad1.08x0.95mm_HandSolder -> Capacitor_SMD:C_0402_1005Metric_Pad0.74x0.62mm_HandSolder
- C3: renamed from C7; footprint Capacitor_SMD:C_0603_1608Metric_Pad1.08x0.95mm_HandSolder -> Capacitor_SMD:C_0402_1005Metric_Pad0.74x0.62mm_HandSolder
- C4: renamed from C8; footprint Capacitor_SMD:C_0603_1608Metric_Pad1.08x0.95mm_HandSolder -> Capacitor_SMD:C_0402_1005Metric_Pad0.74x0.62mm_HandSolder
- C6: renamed from C3; footprint Capacitor_SMD:C_0603_1608Metric_Pad1.08x0.95mm_HandSolder -> Capacitor_SMD:C_0402_1005Metric_Pad0.74x0.62mm_HandSolder
- C7: renamed from C4; footprint Capacitor_SMD:C_0603_1608Metric_Pad1.08x0.95mm_HandSolder -> Capacitor_SMD:C_0402_1005Metric_Pad0.74x0.62mm_HandSolder
- R1: footprint Resistor_SMD:R_0603_1608Metric_Pad0.98x0.95mm_HandSolder -> Resistor_SMD:R_0402_1005Metric_Pad0.72x0.64mm_HandSolder
- R12: renamed from R4; footprint Resistor_SMD:R_0603_1608Metric_Pad0.98x0.95mm_HandSolder -> Resistor_SMD:R_0402_1005Metric_Pad0.72x0.64mm_HandSolder
- R13: renamed from R5; footprint Resistor_SMD:R_0603_1608Metric_Pad0.98x0.95mm_HandSolder -> Resistor_SMD:R_0402_1005Metric_Pad0.72x0.64mm_HandSolder
- R14: renamed from R7; footprint Resistor_SMD:R_0603_1608Metric_Pad0.98x0.95mm_HandSolder -> Resistor_SMD:R_0402_1005Metric_Pad0.72x0.64mm_HandSolder
- R15: renamed from R8; footprint Resistor_SMD:R_0603_1608Metric_Pad0.98x0.95mm_HandSolder -> Resistor_SMD:R_0402_1005Metric_Pad0.72x0.64mm_HandSolder
- R2: renamed from R9; footprint Resistor_SMD:R_0603_1608Metric_Pad0.98x0.95mm_HandSolder -> Resistor_SMD:R_0402_1005Metric_Pad0.72x0.64mm_HandSolder
- R3: renamed from R2; footprint Resistor_SMD:R_0603_1608Metric_Pad0.98x0.95mm_HandSolder -> Resistor_SMD:R_0402_1005Metric_Pad0.72x0.64mm_HandSolder
- R5: renamed from R3; footprint Resistor_SMD:R_0603_1608Metric_Pad0.98x0.95mm_HandSolder -> Resistor_SMD:R_0402_1005Metric_Pad0.72x0.64mm_HandSolder
Connections:
- net GND: now also C10.2, C11.2, C12.2, C5.2, C8.2, C9.1, J2.10, J2.11, J2.12, J2.16, J2.17, J2.18, J2.19, J2.2, J2.20, J2.3, J2.7, J2.8, R11.2, R9.1, U3.2 (GND)
- net I2C_SCL: now also J2.13, R8.1
- net I2C_SDA: now also J2.14, J2.15, R7.1
- net VCC: now also C10.1, C5.1, J2.5, J2.6, L1.1, R4.1, R7.2, R8.2, U3.4 (EN), U3.5 (IN)
- new net: D49.2 (A), L1.2, U3.1 (SW)
- new net: R10.1, R11.1, U3.3 (FB)
- new net: C9.2, J2.22
- new net: J2.21, R9.2
- new net OLED_RST: C8.1, J2.9, R4.2
- new net VPP: C11.1, C12.1, D49.1 (K), J2.23, R10.2
- no-connect marks 20 -> 25
Other:
- note added: "TODO: Add power cut-off circuit"
- moved on the sheet: C1, C13, C14, C15, C2, C3, C4, C6, C7, J1, Q1A, Q1B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

Commit message: Schematic and board progress
Updated gitignore and removed some ignored files
Added power schematic with battery chagrer
Some adjustments to components
Parts:
- removed D1, D10, D11, D12, D13, D14, D15, D16, D17, D18, D19, D2, D20, D21, D22, D23, D24, D25, D26, D27, D28, D29, D3, D30, D31, D32, D33, D34, D35, D36, D37, D38, D39, D4, D40, D41, D42, D43, D44, D45, D46, D47, D48, D5, D6, D7, D8, D9: 1N4148WT, Diode_SMD:D_SOD-523, symbol Diode:1N4148WT
- removed J2: 6871XX183622_687124183622, DataSlice:687124183622, symbol DataSlice:6871XX183622_687124183622
- removed SW1, SW10, SW11, SW12, SW13, SW14, SW15, SW16, SW17, SW18, SW19, SW2, SW20, SW21, SW22, SW23, SW24, SW25, SW26, SW27, SW28, SW29, SW3, SW30, SW31, SW32, SW33, SW34, SW35, SW36, SW37, SW38, SW39, SW4, SW40, SW41, SW42, SW43, SW44, SW45, SW46, SW47, SW48, SW5, SW6, SW7, SW8, SW9: SKRPABE010, SW4_SKRPABE010_ALPS, symbol DataSlice:SKRPABE010
- added C10, C13, C15, C4: 10uF/25V(20%), Capacitor_SMD:C_0402_1005Metric_Pad0.74x0.62mm_HandSolder, symbol Device:C_Small
- added C11, C12, C17, C18: 0.1uF/50V(10%), Capacitor_SMD:C_0402_1005Metric_Pad0.74x0.62mm_HandSolder, symbol Device:C_Small
- added D1, D10, D11, D12, D13, D14, D15, D16, D17, D18, D19, D2, D20, D21, D22, D23, D24, D25, D26, D27, D28, D29, D3, D30, D31, D32, D33, D34, D35, D36, D37, D38, D39, D4, D40, D41, D42, D43, D44, D45, D46, D47, D48, D5, D6, D7, D8, D9: 1N4148WT, Diode_SMD:D_SOD-523, symbol Device:D_Small_Filled
- added D49: 1N5819HW-7-F, Diode_SMD:D_SOD-123, symbol Device:D_Schottky_Small_Filled
- added D50, D51: RED, LED_SMD:LED_0402_1005Metric, symbol Device:LED_Small_Filled
- added J1: USB4105-GF-A, Connector_USB:USB_C_Receptacle_GCT_USB4105-xx-A_16P_TopMnt_Horizontal, symbol Connector:USB_C_Receptacle_USB2.0_16P
- added J2: 68712414522, DataSlice:68712414522, symbol DataSlice:6871XX14522_68712414522
- added J4: 53261-0271, Connector_Molex:Molex_PicoBlade_53261-0271_1x02-1MP_P1.25mm_Horizontal, symbol Connector_Generic:Conn_01x02
- added Q2: FS8205A, Package_SO:TSSOP-8_4.4x3mm_P0.65mm, symbol DataSlice:FS8205A
- added R14: 100R(1%), Resistor_SMD:R_0402_1005Metric_Pad0.72x0.64mm_HandSolder, symbol Device:R_Small
- added R15, R16, R17: 1K(1%), Resistor_SMD:R_0402_1005Metric_Pad0.72x0.64mm_HandSolder, symbol Device:R_Small
- added R18: 3K(1%), Resistor_SMD:R_0402_1005Metric_Pad0.72x0.64mm_HandSolder, symbol Device:R_Small
- added R5, R6: 5.1K(1%), Resistor_SMD:R_0402_1005Metric_Pad0.72x0.64mm_HandSolder, symbol Device:R_Small
- added S_A1, S_AL1, S_AP1, S_B1, S_BS1, S_C1, S_CM1, S_CT1, S_D1, S_DN1, S_E1, S_ES1, S_F1, S_FN1, S_G1, S_H1, S_I1, S_J1, S_K1, S_L1, S_LT1, S_M1, S_MT1, S_N1, S_O1, S_P1, S_PT1, S_Q1, S_R1, S_RI1, S_RT1, S_S1, S_SC1, S_SH1, S_SL1, S_SP1, S_SP2, S_SP3, S_SP4, S_T1, S_TB1, S_U1, S_UP1, S_V1, S_W1, S_X1, S_Y1, S_Z1: SKRPABE010, DataSlice:SW4_SKRPABE010_ALPS, symbol Switch:SW_MEC_5E
- added U3: AMS1117-3.3 / SGM2212-3.3, Package_TO_SOT_SMD:SOT-223-3_TabPin2, symbol Regulator_Linear:AMS1117-3.3
- added U4: DW01A, Package_TO_SOT_SMD:SOT-23-6_Handsoldering, symbol Battery_Management:DW01A
- added U5: TP4056-42-ESOP8, Package_SO:SOIC-8-1EP_3.9x4.9mm_P1.27mm_EP2.41x3.3mm_ThermalVias, symbol Battery_Management:TP4056-42-ESOP8
- C16: renamed from C8; value 100nF/16V(10%) -> 0.1uF/50V(10%)
- C2: renamed from C1; value 10uF/16V(10%) -> 10uF/25V(20%)
- C21: renamed from C6; value 100nF/16V(10%) -> 0.1uF/50V(10%)
- C3: value 10uF/16V(10%) -> 10uF/25V(20%)
- C6: renamed from C2; value 100nF/16V(10%) -> 0.1uF/50V(10%)
- C9: renamed from C4; value 100nF/16V(10%) -> 0.1uF/50V(10%)
- J3: renamed from J1; value Micro_SD_Card_Det2 -> DM3D-SF
- Q1: footprint Package_TO_SOT_SMD:SOT-363_SC-70-6 -> Package_TO_SOT_SMD:SOT-363_SC-70-6_Handsoldering
- R10: renamed from R6; footprint Resistor_SMD:R_0603_1608Metric_Pad0.98x0.95mm_HandSolder -> Resistor_SMD:R_0402_1005Metric_Pad0.72x0.64mm_HandSolder
- U2: value CP2102N-Axx-xQFN28 -> CP2102N-A02-GQFN28
- renumbered C13 to C1, C5 to C14, C9 to C19, C12 to C20, C10 to C22, C11 to C23, C14 to C5, C15 to C7, C7 to C8, D49 to D52, R12 to R1, R7 to R11, R8 to R12, R4 to R13, R9 to R19, R13 to R2, R2 to R20, R10 to R21, R11 to R22, R14 to R3, R1 to R4, R15 to R7, R3 to R8, R5 to R9, SW49 to S_PR1, SW50 to S_RS1, U3 to U6
Connections:
- net GND: now also C10.1, C11.2, C12.2, C13.1, C15.1, C18.2, C4.1, J1.A1 (GND), J1.A12 (GND), J1.B1 (GND), J1.B12 (GND), J1.S1 (SHIELD), J2.10, J2.11, J2.12, J2.16, J2.17, J2.18, J2.19, J2.2, J2.20, J2.3, J2.7, J2.8, Q2.6 (S2), Q2.7 (S2), R16.2, R18.1, R5.2, R6.2, U3.1 (GND), U5.1 (TEMP), U5.3 (GND), U5.9 (EPAD)
- net I2C_SCL: now also J2.13
- net I2C_SDA: now also J2.14, J2.15
- net KB_C_0: now also S_ES1.1, S_ES1.2, S_MT1.1, S_MT1.2, S_SH1.1, S_SH1.2, S_TB1.1, S_TB1.2
- net KB_C_1: now also S_A1.1, S_A1.2, S_CT1.1, S_CT1.2, S_Q1.1, S_Q1.2, S_Z1.1, S_Z1.2
- net KB_C_10: now also S_DN1.1, S_DN1.2, S_P1.1, S_P1.2, S_SC1.1, S_SC1.2, S_SL1.1, S_SL1.2
- net KB_C_11: now also S_AP1.1, S_AP1.2, S_BS1.1, S_BS1.2, S_RI1.1, S_RI1.2, S_RT1.1, S_RT1.2
- net KB_C_2: now also S_AL1.1, S_AL1.2, S_S1.1, S_S1.2, S_W1.1, S_W1.2, S_X1.1, S_X1.2
- net KB_C_3: now also S_C1.1, S_C1.2, S_D1.1, S_D1.2, S_E1.1, S_E1.2, S_FN1.1, S_FN1.2
- net KB_C_4: now also S_F1.1, S_F1.2, S_R1.1, S_R1.2, S_SP1.1, S_SP1.2, S_V1.1, S_V1.2
- net KB_C_5: now also S_B1.1, S_B1.2, S_G1.1, S_G1.2, S_SP2.1, S_SP2.2, S_T1.1, S_T1.2
- net KB_C_6: now also S_H1.1, S_H1.2, S_N1.1, S_N1.2, S_SP3.1, S_SP3.2, S_Y1.1, S_Y1.2
- net KB_C_7: now also S_J1.1, S_J1.2, S_M1.1, S_M1.2, S_SP4.1, S_SP4.2, S_U1.1, S_U1.2
- net KB_C_8: now also S_CM1.1, S_CM1.2, S_I1.1, S_I1.2, S_K1.1, S_K1.2, S_UP1.1, S_UP1.2
- net KB_C_9: now also S_L1.1, S_L1.2, S_LT1.1, S_LT1.2, S_O1.1, S_O1.2, S_PT1.1, S_PT1.2
- net KB_R_0: now also D1.1 (K), D10.1 (K), D11.1 (K), D12.1 (K), D2.1 (K), D3.1 (K), D4.1 (K), D5.1 (K), D6.1 (K), D7.1 (K), D8.1 (K), D9.1 (K)
- net KB_R_1: now also D13.1 (K), D14.1 (K), D15.1 (K), D16.1 (K), D17.1 (K), D18.1 (K), D19.1 (K), D20.1 (K), D21.1 (K), D22.1 (K), D23.1 (K), D24.1 (K)
- net KB_R_2: now also D25.1 (K), D26.1 (K), D27.1 (K), D28.1 (K), D29.1 (K), D30.1 (K), D31.1 (K), D32.1 (K), D33.1 (K), D34.1 (K), D35.1 (K), D36.1 (K)
- net KB_R_3: now also D37.1 (K), D38.1 (K), D39.1 (K), D40.1 (K), D41.1 (K), D42.1 (K), D43.1 (K), D44.1 (K), D45.1 (K), D46.1 (K), D47.1 (K), D48.1 (K)
- net OLED_RST: now also J2.9
- net PC_DN: now also J1.A7 (D-), J1.B7 (D-)
- net PC_DP: now also J1.A6 (D+), J1.B6 (D+)
- net PC_VBUS: now also D49.2 (A), J1.A4 (VBUS), J1.A9 (VBUS), J1.B4 (VBUS), J1.B9 (VBUS)
- net VCC: now also C12.1, C13.2, J2.5, J2.6, U3.2 (VO)
- net VPP: now also J2.23
- net at C19.2: now also J2.22
- net at R19.2: now also J2.21
- new net: D7.2 (A), S_Y1.3 (K), S_Y1.4 (A)
- new net: D32.2 (A), S_M1.3 (K), S_M1.4 (A)
- new net: J1.A5 (CC1), R5.1
- new net: D39.2 (A), S_AL1.3 (K), S_AL1.4 (A)
- new net: D30.2 (A), S_B1.3 (K), S_B1.4 (A)
- new net: D35.2 (A), S_SL1.3 (K), S_SL1.4 (A)
- new net: R18.2, U5.2 (PROG)
- new net: R17.2, U5.6 (~{STDBY})
- new net: R15.1, U5.7 (~{CHRG})
- new net: D12.2 (A), S_BS1.3 (K), S_BS1.4 (A)
- new net: D26.2 (A), S_Z1.3 (K), S_Z1.4 (A)
- new net: D40.2 (A), S_FN1.3 (K), S_FN1.4 (A)
- new net: D28.2 (A), S_C1.3 (K), S_C1.4 (A)
- new net: D1.2 (A), S_ES1.3 (K), S_ES1.4 (A)
- new net: D34.2 (A), S_PT1.3 (K), S_PT1.4 (A)
- new net: D42.2 (A), S_SP2.3 (K), S_SP2.4 (A)
- new net: D14.2 (A), S_A1.3 (K), S_A1.4 (A)
- new net: Q2.4 (G1), U4.1 (OD)
- new net: R16.1, U4.2 (CS)
- new net: Q2.5 (G2), U4.3 (OC)
- new net: C17.1, R14.2, U4.5 (VCC)
- new net: D50.1 (K), R17.1
- new net: D37.2 (A), S_MT1.3 (K), S_MT1.4 (A)
- new net: D29.2 (A), S_V1.3 (K), S_V1.4 (A)
- new net: D46.2 (A), S_LT1.3 (K), S_LT1.4 (A)
- new net: D9.2 (A), S_I1.3 (K), S_I1.4 (A)
- new net: D22.2 (A), S_L1.3 (K), S_L1.4 (A)
- new net: D2.2 (A), S_Q1.3 (K), S_Q1.4 (A)
- new net: D17.2 (A), S_F1.3 (K), S_F1.4 (A)
- new net: D47.2 (A), S_DN1.3 (K), S_DN1.4 (A)
- new net: D51.1 (K), R15.2
- new net: D18.2 (A), S_G1.3 (K), S_G1.4 (A)
- new net: D3.2 (A), S_W1.3 (K), S_W1.4 (A)
- new net: D25.2 (A), S_SH1.3 (K), S_SH1.4 (A)
- new net: D33.2 (A), S_CM1.3 (K), S_CM1.4 (A)
- new net: D44.2 (A), S_SP4.3 (K), S_SP4.4 (A)
- new net: D23.2 (A), S_SC1.3 (K), S_SC1.4 (A)
- new net: D20.2 (A), S_J1.3 (K), S_J1.4 (A)
- new net: D4.2 (A), S_E1.3 (K), S_E1.4 (A)
- new net: D13.2 (A), S_TB1.3 (K), S_TB1.4 (A)
- new net: D15.2 (A), S_S1.3 (K), S_S1.4 (A)
- new net: D41.2 (A), S_SP1.3 (K), S_SP1.4 (A)
- new net: D36.2 (A), S_RT1.3 (K), S_RT1.4 (A)
- new net: D45.2 (A), S_UP1.3 (K), S_UP1.4 (A)
- new net: D31.2 (A), S_N1.3 (K), S_N1.4 (A)
- new net: D38.2 (A), S_CT1.3 (K), S_CT1.4 (A)
- new net: D24.2 (A), S_AP1.3 (K), S_AP1.4 (A)
- new net: D43.2 (A), S_SP3.3 (K), S_SP3.4 (A)
- new net: D5.2 (A), S_R1.3 (K), S_R1.4 (A)
- new net: D21.2 (A), S_K1.3 (K), S_K1.4 (A)
- new net: D48.2 (A), S_RI1.3 (K), S_RI1.4 (A)
- new net: D6.2 (A), S_T1.3 (K), S_T1.4 (A)
- new net: D10.2 (A), S_O1.3 (K), S_O1.4 (A)
- new net: J1.B5 (CC2), R6.1
- new net: Q2.1 (D12), Q2.8 (D12)
- new net: D19.2 (A), S_H1.3 (K), S_H1.4 (A)
- new net: D27.2 (A), S_X1.3 (K), S_X1.4 (A)
- new net: D11.2 (A), S_P1.3 (K), S_P1.4 (A)
- new net: D8.2 (A), S_U1.3 (K), S_U1.4 (A)
- new net: D16.2 (A), S_D1.3 (K), S_D1.4 (A)
- new net +4V: C10.2, C11.1, C15.2, J4.1 (Pin_1), R14.1, U3.3 (VI), U5.5 (BAT)
- new net +5V: C18.1, C4.2, D49.1 (K), D50.2 (A), D51.2 (A), U5.4 (V_{CC}), U5.8 (CE)
- new net -BATT: C17.2, J4.2 (Pin_2), Q2.2 (S1), Q2.3 (S1), U4.6 (GND)
- no-connect marks 25 -> 28
Other:
- moved on the sheet: C1, C14, C16, C19, C2, C20, C21, C22, C23, C3, C5, C6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

Commit message: Board adjustments and some renders
Parts:
- added SW1: K3-1391D-5MM, Button_Switch_SMD:SW_SPDT_PCM12, symbol Switch:SW_SPDT
- J3: renamed from J4; footprint Connector_Molex:Molex_PicoBlade_53261-0271_1x02-1MP_P1.25mm_Horizontal -> Connector_Wire:SolderWire-0.1sqmm_1x02_P3.6mm_D0.4mm_OD1mm
- renumbered J3 to J4, S_BS1 to S1, S_AP1 to S2, S_RT1 to S3, S_RI1 to S4
Connections:
- net +4V: now also SW1.2 (B); no longer J3.1 (Pin_1)
- new net: J3.1 (Pin_1), SW1.1 (A)
Other:
- moved on the sheet: J3

Commit message: CC1101 progress
Parts:
- added C18: 100pF/50V(5%)NP0, Capacitor_SMD:C_0402_1005Metric_Pad0.74x0.62mm_HandSolder, symbol Device:C_Small
- added C20: 0.1uF/50V(10%)X5R, Capacitor_SMD:C_0402_1005Metric_Pad0.74x0.62mm_HandSolder, symbol Device:C_Small
- added C21: 12pF/50V(5%)NP0, Capacitor_SMD:C_0402_1005Metric_Pad0.74x0.62mm_HandSolder, symbol Device:C_Small
- added C22, C27: 1.5pF/50V(5%)NP0, Capacitor_SMD:C_0402_1005Metric_Pad0.74x0.62mm_HandSolder, symbol Device:C_Small
- added C23: 1pF/50V(5%)NP0, Capacitor_SMD:C_0402_1005Metric_Pad0.74x0.62mm_HandSolder, symbol Device:C_Small
- added C24: 47pF/50V(5%)NP0, Capacitor_SMD:C_0402_1005Metric_Pad0.74x0.62mm_HandSolder, symbol Device:C_Small
- added C26: 3.3pF/50V(5%)NP0, Capacitor_SMD:C_0402_1005Metric_Pad0.74x0.62mm_HandSolder, symbol Device:C_Small
- added J5: 66011102111302, Connector_Coaxial:WR-MMCX_Wuerth_66011102111302_Horizontal, symbol Connector:Conn_Coaxial_Small
- added L2, L8: 18nH(5%), Inductor_SMD:L_0402_1005Metric_Pad0.77x0.64mm_HandSolder, symbol Device:L_Small
- added L3, L4, L5, L7: 12nH(5%), Inductor_SMD:L_0402_1005Metric_Pad0.77x0.64mm_HandSolder, symbol Device:L_Small
- added L6: 3.3nH(5%), Inductor_SMD:L_0402_1005Metric_Pad0.77x0.64mm_HandSolder, symbol Device:L_Small
- added R23: 56K(1%), Resistor_SMD:R_0402_1005Metric_Pad0.72x0.64mm_HandSolder, symbol Device:R_Small
- added U6: CC1101RGPR, Package_DFN_QFN:QFN-20-1EP_4x4mm_P0.5mm_EP2.5x2.5mm, symbol DataSlice:CC1101RGPR
- renumbered C21 to C10, C15 to C11, C17 to C12, C18 to C13, C16 to C15, C22 to C16, C23 to C17, C20 to C25, C10 to C28, C11 to C29, C12 to C30, C13 to C31, J4 to J2, J2 to J4, R20 to R10, R10 to R11, R11 to R12, R12 to R13, R13 to R19, R21 to R20, R22 to R21, R19 to R22, U4 to U3, U5 to U4, U6 to U5, U3 to U7
Connections:
- net SPI_CK: now also U6.1 (SCLK)
- net SPI_DI: now also U6.2 (SO(GDO1))
- net SPI_DO: now also U6.20 (SI)
- new net: C26.1, L4.2, L5.1
- new net: C21.2, J5.1 (In), L6.1
- new net: C24.2, L6.2
- new net: C23.2, C27.1, L7.1, L8.2
- new net: L7.2, U6.13 (RF_N)
- new net: L3.1, U6.12 (RF_P)
- new net: C22.1, C23.1, L2.1, L3.2
- new net: C22.2, L4.1, L8.1
- new net: C21.1, C24.1, L5.2
- new net: R23.1, U6.17 (RBIAS)
- new net: C20.1, U6.5 (DCOUPL)
- new net: C18.1, L2.2
- new net GNDA: C18.2, C20.2, C26.2, C27.2, J5.2 (Ext), R23.2, U6.16 (GND_16), U6.19 (GND_19), U6.21 (EXP)
- new net VDDA: U6.11 (AVDD_11), U6.14 (AVDD_14), U6.15 (AVDD_15), U6.18 (DGUARD), U6.4 (DVDD), U6.9 (AVDD_9)
Other:
- moved on the sheet: C10, C11, C12, C13, C14, C15, C16, C17, C19, C25, C28, C29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

Commit message: Added USB host and finished CC1110 schematic
Parts:
- added C16: 1uF/50V(10%), Capacitor_SMD:C_0402_1005Metric_Pad0.74x0.62mm_HandSolder, symbol Device:C_Small
- added C19: 0.1uF/50V(10%), Capacitor_SMD:C_0402_1005Metric_Pad0.74x0.62mm_HandSolder, symbol Device:C_Small
- added C29, C35: 12pF/50V(5%)NP0, Capacitor_SMD:C_0402_1005Metric_Pad0.74x0.62mm_HandSolder, symbol Device:C_Small
- added D53: 1N5819HW-7-F, Diode_SMD:D_SOD-123, symbol Device:D_Schottky_Small_Filled
- added J5: USB4105-GF-A, Connector_USB:USB_C_Receptacle_GCT_USB4105-xx-A_16P_TopMnt_Horizontal, symbol Connector:USB_C_Receptacle_USB2.0_16P
- added R20, R21: 5.1K(1%), Resistor_SMD:R_0402_1005Metric_Pad0.72x0.64mm_HandSolder, symbol Device:R_Small
- added Y1: 3225-26M-SR, Crystal:Crystal_SMD_3225-4Pin_3.2x2.5mm_HandSoldering, symbol Device:Crystal_GND24_Small
- renumbered C16 to C17, C17 to C18, C18 to C20, C19 to C21, C20 to C22, C21 to C23, C22 to C24, C23 to C25, C24 to C26, C25 to C27, C26 to C28, C27 to C30, C28 to C31, C29 to C32, C30 to C33, C31 to C34, J5 to J6, R20 to R22, R21 to R23, R22 to R24, R23 to R25
Connections:
- net +4V: now also D53.2 (A)
- net GND: now also J5.A1 (GND), J5.A12 (GND), J5.B1 (GND), J5.B12 (GND), J5.S1 (SHIELD)
- net GNDA: now also C16.1, C19.2, C29.2, C35.2
- net HOST_DN: now also J5.A7 (D-), J5.B7 (D-)
- net HOST_DP: now also J5.A6 (D+), J5.B6 (D+)
- net VDDA: now also C16.2, C19.1
- net at U6.10 (XOSC_Q2): now also C35.1, Y1.1
- net SUB_CS: now reaches U6.7 (CSN)
- net SUB_CS: now also U1.33 (IO40)
- net at U6.8 (XOSC_Q1): now also C29.1, Y1.3
- new net: D53.1 (K), J5.A4 (VBUS), J5.A9 (VBUS), J5.B4 (VBUS), J5.B9 (VBUS), R20.1, R21.1
- new net: J5.A5 (CC1), R20.2
- new net: J5.B5 (CC2), R21.2
- no-connect marks 28 -> 32
Other:
- note added: "TODO: Add USB protection"
- note added: "TODO: Add switch between 868 and 433 MHz, currently supporting only 868 MHz"
- moved on the sheet: C20, C22, C23, C24, C25, C26, C28, C30, J6, L2, L3, L4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

Commit message: ERC correction
Parts:
- added R25, R26: 0R, Jumper:SolderJumper-2_P1.3mm_Open_RoundedPad1.0x1.5mm, symbol Device:R_Small
- renumbered R25 to R27
Connections:
- net GND: now also R26.2
- net GNDA: now also R26.1
- net VCC: now also R25.2
- net VDDA: now also R25.1
- net +4V renamed +BATT
- no-connect marks 32 -> 35
Other:
- moved on the sheet: C22
