File: DataSliceHW/DataSliceHW.kicad_sch (KiCad schematic)
At the start: 190 parts, among them J1 USB4105-GF-A, J2 DM3D-SF, J3 53261-0271, J4 68712414522, J5 USB4105-GF-A, J6 66011102111302, Q1 BC847BDW1, Q2 FS8205A, SW1 K3-1391D-5MM, U1 ESP32-S3-WROOM-1, U2 CP2102N-A02-GQFN28, U3 DW01A, U4 TP4056-42-ESOP8, U5 MT3608/SX1308, U6 CC1101RGPR, U7 AMS1117-3.3 / SGM2212-3.3, Y1 3225-26M-SR

Commit message: Minor schematic changes and some PCB tracing progress
Parts:
- removed C12: 0.1uF/50V(10%), Capacitor_SMD:C_0402_1005Metric_Pad0.74x0.62mm_HandSolder, symbol Device:C_Small
- removed Q2: FS8205A, Package_SO:TSSOP-8_4.4x3mm_P0.65mm, symbol DataSlice:FS8205A
- removed R14: 100R(1%), Resistor_SMD:R_0402_1005Metric_Pad0.72x0.64mm_HandSolder, symbol Device:R_Small
- removed R16: 1K(1%), Resistor_SMD:R_0402_1005Metric_Pad0.72x0.64mm_HandSolder, symbol Device:R_Small
- removed U3: DW01A, Package_TO_SOT_SMD:SOT-23-6_Handsoldering, symbol Battery_Management:DW01A
- C1, C5, C8: value 1uF/16V(10%) -> 1uF(10%)
- C10: renamed from C31; value 10uF/25V(20%) -> 10uF(20%)
- C11: renamed from C32; value 0.1uF/50V(10%) -> 0.1uF(10%)
- C12: renamed from C33; value 0.1uF/50V(10%) -> 0.1uF(10%)
- C13: renamed from C34; value 10uF/25V(20%) -> 10uF(20%)
- C14: renamed from C10; value 0.1uF/50V(10%) -> 0.1uF(10%)
- C15: renamed from C13; value 0.1uF/50V(10%) -> 0.1uF(10%)
- C16: renamed from C11; value 10uF/25V(20%) -> 10uF(20%)
- C17: renamed from C14; value 4.7uF/16V(10%) -> 4.7uF(10%)
- C19: renamed from C15; value 0.1uF/50V(10%) -> 0.1uF(10%)
- C2, C3, C4: value 10uF/25V(20%) -> 10uF(20%)
- C21: renamed from C17; value 22uF/50V(10%) -> 22uF(10%)
- C22: renamed from C18; value 22uF/50V(10%) -> 22uF(10%)
- C23: renamed from C20; value 100pF/50V(5%)NP0 -> 100pF(5%)NP0
- C24: renamed from C22; value 0.1uF/50V(10%)X5R -> 0.1uF(10%)X5R
- C25: renamed from C23; value 12pF/50V(5%)NP0 -> 12pF(5%)NP0
- C26: renamed from C24; value 1.5pF/50V(5%)NP0 -> 1.5pF(5%)NP0
- C27: renamed from C21; value 4.7uF/50V(10%) -> 4.7uF(10%)
- C28: renamed from C25; value 1pF/50V(5%)NP0 -> 1pF(5%)NP0
- C29: renamed from C26; value 47pF/50V(5%)NP0 -> 47pF(5%)NP0
- C30: renamed from C28; value 3.3pF/50V(5%)NP0 -> 3.3pF(5%)NP0
- C31: renamed from C29; value 12pF/50V(5%)NP0 -> 12pF(5%)NP0
- C32: renamed from C27; value 4.7uF/50V(10%) -> 4.7uF(10%)
- C33: renamed from C30; value 1.5pF/50V(5%)NP0 -> 1.5pF(5%)NP0
- C34: renamed from C35; value 12pF/50V(5%)NP0 -> 12pF(5%)NP0
- C6, C9: value 0.1uF/50V(10%) -> 0.1uF(10%)
- C7: value 4.7uF/16V(10%) -> 4.7uF(10%)
- D50: value RED -> BLUE
- renumbered C16 to C18, C19 to C20, J6 to J5, J5 to J6, R17 to R14, R18 to R16, R19 to R17, R20 to R18, R21 to R19, R22 to R20, R23 to R21, R24 to R22, R25 to R23, R26 to R24, R27 to R25, U7 to U3
Connections:
- net -BATT is gone; now on net GND: J3.2 (Pin_2)
- net +5V: now also C15.2; no longer C15.1
- net GND: now also C15.1, R16.2; no longer C15.2, R16.1
- net GNDA: now also C34.1; no longer C34.2
- net KB_C_0: now also U1.15 (IO3); no longer U1.39 (IO1)
- net KB_C_1: now also U1.16 (IO46); no longer U1.38 (IO2)
- net KB_C_10: now also U1.39 (IO1); no longer U1.8 (IO15)
- net KB_C_11: now also U1.38 (IO2); no longer U1.9 (IO16)
- net KB_C_2: now also U1.17 (IO9); no longer U1.15 (IO3)
- net KB_C_3: now also U1.12 (IO8); no longer U1.4 (IO4)
- net KB_C_4: now also U1.9 (IO16); no longer U1.5 (IO5)
- net KB_C_5: now also U1.8 (IO15); no longer U1.6 (IO6)
- net KB_C_7: now also U1.6 (IO6); no longer U1.12 (IO8)
- net KB_C_8: now also U1.5 (IO5); no longer U1.17 (IO9)
- net KB_C_9: now also U1.4 (IO4); no longer U1.22 (IO14)
- net KB_R_0: now also U1.22 (IO14); no longer U1.26 (IO45)
- net KB_R_1: now also U1.24 (IO47); no longer U1.16 (IO46)
- net KB_R_2: now also U1.25 (IO48); no longer U1.24 (IO47)
- net KB_R_3: now also U1.26 (IO45); no longer U1.25 (IO48)
- net HOST_VBUS: now reaches D53.1 (K), J6.A4 (VBUS), J6.A9 (VBUS), J6.B4 (VBUS), J6.B9 (VBUS), R18.1, R19.1
- net at U6.10 (XOSC_Q2), Y1.1: now also C34.2; no longer C34.1
- net at U4.2 (PROG): now also R16.1; no longer R16.2
- net at U4.7 (~{CHRG}): now also R15.2; no longer R15.1
- net +4V: now reaches J3.1 (Pin_1), SW1.1 (A)
- net at D51.1 (K): now also R15.1; no longer R15.2
- no-connect marks 35 -> 34
Other:
- moved on the sheet: C10, C11, C12, C13, C15, C16, C18, C20, C23, C24, C25, C26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

Commit message: Finalized firt prototype Completed PCB design Finalized schematic
Parts:
- removed C28: 1pF(5%)NP0, Capacitor_SMD:C_0402_1005Metric_Pad0.74x0.62mm_HandSolder, symbol Device:C_Small
- removed L3, L7: 12nH(5%), Inductor_SMD:L_0402_1005Metric_Pad0.77x0.64mm_HandSolder, symbol Device:L_Small
- removed L6: 3.3nH(5%), Inductor_SMD:L_0402_1005Metric_Pad0.77x0.64mm_HandSolder, symbol Device:L_Small
- added J4: Conn_01x04, Connector_PinHeader_2.54mm:PinHeader_1x04_P2.54mm_Horizontal, symbol Connector_Generic:Conn_01x04
- added J5: Conn_01x02, Connector_PinHeader_2.54mm:PinHeader_1x02_P2.54mm_Horizontal, symbol Connector_Generic:Conn_01x02
- added J9: Conn_01x05, Connector_PinSocket_2.54mm:PinSocket_1x05_P2.54mm_Vertical, symbol Connector_Generic:Conn_01x05
- C24: renamed from C23; value 100pF(5%)NP0 -> 220pF(5%)NP0
- C25: renamed from C26; value 1.5pF(5%)NP0 -> 3.9pF(5%)NP0
- C27: renamed from C25; value 12pF(5%)NP0 -> 220pF(5%)NP0
- C28: renamed from C30; value 3.3pF(5%)NP0 -> 8.2pF(5%)NP0
- C29: value 47pF(5%)NP0 -> 5.6pF(5%)NP0
- C31: renamed from C33; value 1.5pF(5%)NP0 -> 3.9pF(5%)NP0
- L2: value 18nH(5%) -> 27nH(5%)
- L3: renamed from L4; value 12nH(5%) -> 22nH(5%)
- L4: renamed from L5; value 12nH(5%) -> 27nH(5%)
- L5: renamed from L8; value 18nH(5%) -> 27nH(5%)
- Y1: footprint Crystal:Crystal_SMD_3225-4Pin_3.2x2.5mm_HandSoldering -> Crystal:Crystal_SMD_3225-4Pin_3.2x2.5mm
- renumbered C24 to C23, C27 to C26, C32 to C30, C34 to C32, C31 to C33, J4 to J6, J6 to J7, J5 to J8
Connections:
- net GND: now also J6.Z1, J6.Z2, J5.2 (Pin_2), J9.5 (Pin_5)
- net GNDA: now also C29.1, Y1.2, Y1.4
- net RS_RX: now also J9.2 (Pin_2)
- net RS_TX: now also J9.1 (Pin_1)
- net SPI_CK: now also J4.3 (Pin_3)
- net SPI_CS: now also J4.1 (Pin_1)
- net SPI_DI: now also J4.2 (Pin_2)
- net SPI_DO: now also J4.4 (Pin_4)
- net VCC: now also J5.1 (Pin_1), J9.4 (Pin_4)
- net at C29.2: now also C27.1, L4.2
- net at C31.1, L5.2: now also U6.13 (RF_N)
- net at U6.12 (RF_P): now also C25.1, L2.1
- no-connect marks 34 -> 31
Other:
- note added: "TODO: Add switch between 868 and 433 MHz, currently supporting only 433 MHz"
- note added: "TODO: Use SY7088 for Bat-to-5V"
- note added: "TODO: Use SY8089"
- note added: "TODO: Use TP4057"
- note removed: "TODO: Add switch between 868 and 433 MHz, currently supporting only 868 MHz"
- moved on the sheet: C18, C20, C23, C24, C25, C27, C28, C29, C31, C32, C33, J8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

Commit message: Minor PCB changes
Parts:
- removed R23, R24: 0R, Jumper:SolderJumper-2_P1.3mm_Open_RoundedPad1.0x1.5mm, symbol Device:R_Small
- renumbered R25 to R23
Connections:
- net GNDA is gone; now on net GND: C18.1, C20.2, C23.2, C24.2, C28.2, C29.1, C31.2, C32.1, C33.2, J8.2 (Ext), R23.2, U6.16 (GND_16), U6.19 (GND_19), U6.21 (EXP), Y1.2, Y1.4
- net VDDA is gone; now on net VCC: C18.2, C20.1, U6.11 (AVDD_11), U6.14 (AVDD_14), U6.15 (AVDD_15), U6.18 (DGUARD), U6.4 (DVDD), U6.9 (AVDD_9)
